Commit message: update urdf

File: z1_description/urdf/z1.urdf.xacro (robot description, xacro)
@@ -278,5 +278,5 @@
         </link>
         <joint name="jointGripper" type="fixed">
-            <origin  xyz="0.0905 0 0" rpy="0 0 0" />
+            <origin  xyz="0.1205 0 0" rpy="0 0 0" />
             <parent link="gripper_base" />
             <child link="gripper_link" />
@@ -286,6 +286,6 @@
             <inertial>
             <origin
-                xyz="7.3899220076612E-16 1.73472347597681E-17 0.0112170244662773"
-                rpy="0 0 0" />
+                xyz="-0.03 1.73472347597681E-17 0.0112170244662773"
+                rpy="1.5708 0 1.5708" />
             <mass
                 value="0.0538139787320802" />
@@ -299,5 +299,5 @@
             </inertial>
             <visual>
-                <origin xyz="0 0 0" rpy="1.5708 0 1.5708" />
+                <origin xyz="-0.03 0 0" rpy="1.5708 0 1.5708" />
                 <geometry>
                     <mesh filename="package://z1_description/meshes/collision/gripper_link.STL" />
@@ -308,5 +308,5 @@
             </visual>
             <collision>
-                <origin xyz="0 0 0" rpy="1.5708 0 1.5708" />
+                <origin xyz="-0.03 0 0" rpy="1.5708 0 1.5708" />
                 <geometry>
                     <mesh filename="package://z1_description/meshes/collision/gripper_link.STL" />
@@ -330,5 +330,6 @@
         </link>
         <joint name="camera_joint" type="fixed">
-            <origin rpy="-1.6034 -0.0629 -1.5489" xyz="-0.0718 0.0494 0.0932" />
+            <!-- <origin rpy="-1.6034 -0.0629 -1.5489" xyz="-0.0718 0.0494 0.0932" /> -->
+            <origin rpy="-1.5881 -0.0244 -1.5670" xyz="-0.0949 0.0345 0.0879" />
             <parent link="gripper_link" />
             <child link="camera_link" />

Commit message: adapt to orbbec camera and replace z1_hardware_interface with move_group to control z1

File: z1_description/urdf/z1.urdf.xacro (robot description, xacro)
@@ -331,5 +331,5 @@
         <joint name="camera_joint" type="fixed">
             <!-- <origin rpy="-1.6034 -0.0629 -1.5489" xyz="-0.0718 0.0494 0.0932" /> -->
-            <origin rpy="-1.5881 -0.0244 -1.5670" xyz="-0.0949 0.0345 0.0879" />
+            <origin rpy="-1.5860 -0.0219 -1.5744" xyz="-0.0943 0.0218 0.0898" />
             <parent link="gripper_link" />
             <child link="camera_link" />
